Commit message: Enviroment definition

File: urdf/giraffe.urdf (robot description, URDF)
Before this commit: robot giraffe_robot, 7 links, 6 joints
Links:
- added link ceiling; visual box size=5 12 0.1
- added link floor; visual box size=5 12 0.1
Joints:
- removed joint world_joint
- added joint base_link_fixed: type fixed, parent ceiling, child base_link, origin xyz=0.0 0.0 0.0 rpy=0.0 0.0 0.0
- added joint ceiling_fixed: type fixed, parent floor, child ceiling, origin xyz=0 0 4.05 rpy=0 0 0
- added joint floor_fixed: type fixed, parent world, child floor, origin xyz=2.5 6 0 rpy=0 0 0

Commit message: Uodate the robot architecture

File: urdf/giraffe.urdf (robot description, URDF)
Before this commit: robot giraffe_robot, 9 links, 8 joints
Links:
- removed link mic_pitch_link
- removed link yaw_link
- added link forearm_link; visual cylinder length=0.06 radius=0.03; visual cylinder length=0.06 radius=0.03
- added link mic; visual cylinder length=0.15 radius=0.02
- added link shoulder_link; visual cylinder length=0.1 radius=0.05
- link base_link: mass None -> 4.0; geometry collision mesh filename=package://ur_description/meshes/ur5/collision/base.stl; visual mesh filename=package://ur_description/meshes/ur5/collision/base.stl
- link extend_link: geometry visual cylinder length=4.5 radius=0.03
- link mic_link: geometry visual cylinder length=0.15 radius=0.01
- link pitch_link: geometry visual box size=0.2 0.1 0.1; visual cylinder length=0.1 radius=0.05
Joints:
- removed joint extend_joint
- removed joint mic_pitch_joint
- removed joint pitch_joint
- removed joint yaw_joint
- added joint mic_fixed: type fixed, parent mic_link, child mic, origin xyz=0.15 0 0 rpy=0 ${pi_2} 0
- added joint mic_yaw_joint: type revolute, parent forearm_link, child mic_link, origin xyz=1.03 0 0 rpy=-${pi_2} 0 -${pi_2}, axis 0 0 1, limit lower=-3.14 upper=3.14 effort=5 velocity=1.0
- added joint prismatic_joint: type prismatic, parent pitch_link, child extend_link, origin xyz=2.4 0.1 0 rpy=0 ${pi_2} 0, axis 0 0 1, limit lower=0 upper=4 effort=50 velocity=0.5
- added joint shoulder_pitch_joint: type revolute, parent shoulder_link, child pitch_link, origin xyz=0.0 0.0 0.0 rpy=${pi_2} 0.0 0.0, axis 0 0 1, limit lower=0 upper=${pi} effort=150.0 velocity=3.15
- added joint shoulder_yaw_joint: type revolute, parent base_link, child shoulder_link, origin xyz=0.0 0.0 0.1 rpy=0 0 0, axis 0 0 1, limit lower=-${pi} upper=${pi} effort=50.0 velocity=1.5
- joint base_link_fixed: origin xyz=0.0 0.0 0.0 rpy=0.0 0.0 0.0 -> xyz=2.5 6 4 rpy=${pi} 0 ${pi_2}; parent ceiling -> world
- joint mic_roll_joint: child mic_link -> forearm_link; limit lower=-3.14 upper=3.14 effort=5 velocity=1.0 -> lower=-1.57 upper=1.57 effort=5 velocity=1.0; origin xyz=0 0 -0.3 rpy=0 0 0 -> xyz=0 0 0.2 rpy=${pi} -${pi_2} 0; parent mic_pitch_link -> extend_link

Commit message: Update robot urdf

File: urdf/giraffe.urdf (robot description, URDF)
Before this commit: robot giraffe_robot, 10 links, 9 joints
Links:
- removed link forearm_link
- removed link pitch_link
- added link arm_link; visual box size=0.2 0.1 0.1; visual cylinder length=${arm_length + shoulder_joint_radius} radius=${arm_radius}
- added link wrist_link; visual cylinder length=${wrist_link_length} radius=${wrist_radius}; visual cylinder length=${wrist_radius*2} radius=${wrist_radius}
- link base_link: mass 4.0 -> None; geometry collision cylinder length=0 radius=${base_radius}; visual cylinder length=0 radius=${base_radius}
- link extend_link: geometry visual cylinder length=${prismatic_travel + wrist_radius} radius=${wrist_radius}
- link shoulder_link: geometry visual cylinder length=${shoulder_joint_height} radius=${shoulder_joint_radius}
Joints:
- removed joint shoulder_pitch_joint
- removed joint shoulder_yaw_joint
- added joint shoulder_pitch: type revolute, parent shoulder_link, child arm_link, origin xyz=0.0 0.0 0.0 rpy=-${pi_2} 0.0 0.0, axis 0 0 1, limit lower=-${pi} upper=0 effort=150.0 velocity=3.15
- added joint shoulder_yaw: type revolute, parent base_link, child shoulder_link, origin xyz=0 0 ${shoulder_joint_height} rpy=0 0 0, axis 0 0 1, limit lower=-${pi} upper=${pi} effort=50 velocity=1.5
- joint mic_roll_joint: child forearm_link -> wrist_link; origin xyz=0 0 0.2 rpy=${pi} -${pi_2} 0 -> xyz=0 0 0 rpy=${pi} -${pi_2} 0
- joint mic_yaw_joint: parent forearm_link -> wrist_link
- joint prismatic_joint: limit lower=0 upper=4 effort=50 velocity=0.5 -> lower=0 upper=${prismatic_travel} effort=50 velocity=0.5; origin xyz=2.4 0.1 0 rpy=0 ${pi_2} 0 -> xyz=${arm_length + shoulder_joint_radius + wrist_radius} -${prismatic_height_delta} 0 rpy=-${pi_2} 0 -${pi_2}; parent pitch_link -> arm_link

Commit message: first attemption definition direct kinematics

File: urdf/giraffe.urdf (robot description, URDF)
Before this commit: robot giraffe_robot, 10 links, 9 joints
Links:
- removed link mic_link
- added link mic-link; visual cylinder length=${mic_stick_length} radius=${mic_stick_radius}
- link mic: geometry visual sphere radius=${mic_stick_radius}
- link wrist_link: geometry visual cylinder length=${wrist_link_length} radius=${wrist_radius}; visual cylinder length=${wrist_radius*2} radius=${wrist_radius}
Joints:
- removed joint mic_fixed
- removed joint mic_roll_joint
- removed joint shoulder_pitch
- added joint mic_pitch_joint: type revolute, parent wrist_link, child mic-link, origin xyz=0 0 ${wrist_link_length - wrist_radius} rpy=-${pi_2} 0 -${pi_2}, axis 0 0 1, limit lower=-3.14 upper=3.14 effort=5 velocity=1.0
- added joint mic_stick_joint: type fixed, parent mic-link, child mic, origin xyz=${mic_stick_length + wrist_radius + mic_stick_radius} 0 0 rpy=0 0 0
- added joint shoulder_roll: type revolute, parent shoulder_link, child arm_link, origin xyz=0.0 0.0 0.0 rpy=-${pi_2} 0.0 0.0, axis 0 0 1, limit lower=-${pi} upper=0 effort=150.0 velocity=3.15
- joint base_link_fixed: origin xyz=2.5 6 4 rpy=${pi} 0 ${pi_2} -> xyz=2.5 6 4 rpy=${pi} 0 -${pi_2}
- joint mic_yaw_joint: child mic_link -> wrist_link; limit lower=-3.14 upper=3.14 effort=5 velocity=1.0 -> lower=-1.57 upper=1.57 effort=5 velocity=1.0; origin xyz=1.03 0 0 rpy=-${pi_2} 0 -${pi_2} -> xyz=0 0 0 rpy=${pi} -${pi_2} 0; parent wrist_link -> extend_link

Commit message: Defined the Inertia

File: urdf/giraffe.urdf (robot description, URDF)
Before this commit: robot giraffe_robot, 10 links, 9 joints
Links:
- link arm_link: mass None -> ${arm_mass}; geometry visual box size=0.2 0.1 0.1; visual cylinder length=${arm_length + shoulder_joint_radius} radius=${arm_radius}
- link base_link: geometry visual cylinder length=0 radius=${base_radius}
- link extend_link: mass None -> ${extend_link_mass}; geometry visual cylinder length=${extend_link_length} radius=${wrist_radius}
- link mic: mass None -> ${mic_stick_mass}
- link mic_link: mass None -> ${mic_stick_mass}
- link shoulder_link: mass None -> ${2 * shoulder_joint_mass}; geometry visual cylinder length=${shoulder_joint_height} radius=${shoulder_joint_radius}; visual cylinder length=${shoulder_joint_height} radius=${shoulder_joint_radius}
- link wrist_link: mass None -> ${wrist_link_mass}
