Commit message: Define and tested Direct Kinematics

File: urdf/giraffe_processed.urdf (robot description, URDF)
Before this commit: robot giraffe_robot, 10 links, 9 joints
Links:
- link arm_link: geometry visual box size=0.2 0.1 0.1; visual cylinder length=0.1 radius=0.05
- link base_link: geometry collision cylinder length=0 radius=0.1; visual cylinder length=0 radius=0.1
- link extend_link: geometry visual cylinder length=4.025 radius=0.025
- link mic: geometry visual sphere radius=0.015
- link mic_link: geometry visual cylinder length=0.15 radius=0.015
- link shoulder_link: geometry visual cylinder length=0.1 radius=0.05
- link wrist_link: geometry visual cylinder length=0.05 radius=0.025; visual cylinder length=0.05 radius=0.025
Joints:
- joint base_link_fixed: origin xyz=2.5 6 4 rpy=${pi} 0 -${pi_2} -> xyz=2.5 6 4 rpy=3.141592653589793 0 -1.5707963267948966
- joint mic_pitch_joint: origin xyz=0 0 ${wrist_link_length - wrist_radius} rpy=-${pi_2} 0 -${pi_2} -> xyz=0 0 0.975 rpy=-1.5707963267948966 0 -1.5707963267948966
- joint mic_stick_joint: origin xyz=${mic_stick_length + wrist_radius + (2*mic_stick_radius)} 0 0 rpy=0 0 0 -> xyz=0.205 0 0 rpy=0 0 0
- joint mic_yaw_joint: origin xyz=0 0 0 rpy=${pi} -${pi_2} 0 -> xyz=0 0 0 rpy=3.141592653589793 -1.5707963267948966 0
- joint prismatic_joint: limit lower=0 upper=${prismatic_travel} effort=50 velocity=0.5 -> lower=0 upper=4.0 effort=50 velocity=0.5; origin xyz=${arm_length + shoulder_joint_radius + wrist_radius} -${prismatic_height_delta} 0 rpy=-${pi_2} 0 -${pi_2} -> xyz=2.4749999999999996 -0.1 0 rpy=-1.5707963267948966 0 -1.5707963267948966
- joint shoulder_roll: limit lower=-${pi} upper=0 effort=150.0 velocity=3.15 -> lower=-3.141592653589793 upper=0 effort=150.0 velocity=3.15; origin xyz=0.0 0.0 0.0 rpy=-${pi_2} 0.0 0.0 -> xyz=0.0 0.0 0.0 rpy=-1.5707963267948966 0.0 0.0
- joint shoulder_yaw: limit lower=-${pi} upper=${pi} effort=50 velocity=1.5 -> lower=-3.141592653589793 upper=3.141592653589793 effort=50 velocity=1.5; origin xyz=0 0 ${shoulder_joint_height} rpy=0 0 0 -> xyz=0 0 0.1 rpy=0 0 0

Commit message: defined ForwardKinematics

File: urdf/giraffe_processed.urdf (robot description, URDF)
Before this commit: robot giraffe_robot, 10 links, 9 joints
Links:
- link arm_link: mass None -> 50.89380098815466; geometry visual box size=0.2 0.1 0.1; visual cylinder length=2.4499999999999997 radius=0.05
- link base_link: geometry visual cylinder length=0 radius=0.1
- link extend_link: mass None -> 21.33828635180443
- link mic: mass None -> 0.2862776305583699
- link mic_link: mass None -> 0.2862776305583699
- link shoulder_link: mass None -> 4.2411500823462225; geometry visual cylinder length=0.1 radius=0.05; visual cylinder length=0.1 radius=0.05
- link wrist_link: mass None -> 5.831581363226055
